File: raspnixie.sch (EAGLE design)
At the start: 30 parts, among them IC1 74141N, IC2 74141N, IC3 74141N, IC4 74141N, T1 IRF644B, T2 13001, U1 ZM1000, U2 ZM1000, U3 ZM1000, U4 ZM1000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

Commit message: mark. 14
Parts:
- removed C2: 10n, rcl:C-EUC0603
- removed CONNECTME: 0, rcl:R-EU_R0805
- removed R2: 1M5, rcl:R-EU_0613/15
- removed RN1: 10M, resistor-dil:4R-N0603-ARC
- removed RN6: 18k, resistor-dil:4R-N0603-ARV
- added C8: 10n, rcl:C-EUC1206K
- added JP1: (no value), jumper:JP1Q
- added R10, R11, R12, R9: 10M, rcl:R-EU_R1206
- added R2A, R2B: 750k, rcl:R-EU_R1206
- added R5, R6, R7, R8: 15k, rcl:R-EU_R1206
- C3, C5, C6, C7: device rcl:C-EUC0603 -> rcl:C-EUC1206K
- L1: value 101 -> 221; device raspnixie:WHC1050 -> raspnixie:WHC1770
- R1, R3, R4: device rcl:R-EU_R0603 -> rcl:R-EU_R1206
- RSENSE: device raspnixie:CEMENT_RESISTOR -> rcl:R-EU_R2010
- VR1: device pot:TRIM_EU-S64W -> pot-hex:TRIM_EU-S64W-ROUND
- X1: value RASPI_BOARD_B+#_E3P -> RASPI_BOARD_B+#_E3; device raspberrypi_bastelstube_v13:RASPI_BOARD_B+#_E3P -> raspberrypi_bastelstube_v13:RASPI_BOARD_B+#_E3
- renumbered U5 to IC5
Connections:
- new net N$75: R2A.2, R2B.1
- net GND: now also C8.2, R10.2, R11.2, R12.2, R9.2; no longer C2.2, RN1A.2, RN1B.2, RN1C.2, RN1D.2
- net N$1: now also R9.1; no longer RN1A.1
- net N$2: now also R10.1; no longer RN1B.1
- net N$3: now also R11.1; no longer RN1C.1
- net N$4: now also R12.1; no longer RN1D.1
- net N$65: now also R5.1; no longer RN6A.1
- net N$66: now also R6.1; no longer RN6B.1
- net N$70: now also R2A.1; no longer R2.2
- net N$71: now also R7.1; no longer RN6C.1
- net N$72: now also R8.1; no longer RN6D.1
- net V+: now also JP1.1; no longer CONNECTME.2, IC5.V+
- net VCC: now also C8.1, IC5.V+, JP1.2; no longer C2.1, CONNECTME.1
- net VH: now also R2B.2, R5.2, R6.2, R7.2, R8.2; no longer R2.1, RN6A.2, RN6B.2, RN6C.2, RN6D.2
Other:
- moved on the sheet: C5, C6, C7

Commit message: steal from other libraries
Parts:
- IC1, IC2, IC3, IC4: device 74xx-eu:74141N -> raspnixie:74141N
- IC5: device MAX1771CPA:MAX1771CPA+ -> raspnixie:MAX1771CPA+
- T1: device Transistor:NMOSFET_TO220 -> transistor-power:IRF540
- T2: value 13001 -> A42; device Transistor:NPN_TO92 -> transistor:-NPN-TO92
- VR1: device pot-hex:TRIM_EU-S64W-ROUND -> raspnixie:TRIM_EU-S64W-ROUND
- X1: device raspberrypi_bastelstube_v13:RASPI_BOARD_B+#_E3 -> raspnixie:RASPI_BOARD_B+#_E3

Commit message: 2021-06-07 Mk.16
Parts:
- added C2: 100n, rcl:C-EUC1206K
- IC5: value MAX1771CPA+ -> MAX1771CPA+SO08; device raspnixie:MAX1771CPA+ -> raspnixie:MAX1771CPA+SO08
Connections:
- net GND: now also C2.2
- net VCC: now also C2.1
Other:
- moved on the sheet: C1
Changed lines of the file:
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@@
 <?xml version="1.0" encoding="utf-8"?>
 <!DOCTYPE eagle SYSTEM "eagle.dtd">
-<eagle version="9.6.0">
+<eagle version="9.6.2">
 <drawing>
 <settings>
@@
 </variantdefs>
 <classes>
-<class number="0" name="default" width="0" drill="0">
+<class number="0" name="default" width="0.1524" drill="0.3">
+<clearance class="0" value="0.1524"/>
 </class>
 <class number="1" name="power" width="1.397" drill="0.635">
+<clearance class="0" value="0.508"/>
 <clearance class="1" value="0.508"/>
 </class>
@@
 <part name="IC4" library="raspnixie" deviceset="74*141" device="N" package3d_urn="urn:adsk.eagle:package:922/2"/>
 <part name="U4" library="raspnixie" deviceset="ZM1000" device=""/>
-<part name="IC5" library="raspnixie" deviceset="MAX1771CPA+" device=""/>
+<part name="IC5" library="raspnixie" deviceset="MAX1771CPA+" device="SO08"/>
 <part name="P+2" library="supply1" library_urn="urn:adsk.eagle:library:371" deviceset="VCC" device=""/>
 <part name="C3" library="rcl" library_urn="urn:adsk.eagle:library:334" deviceset="C-EU" device="C1206K" package3d_urn="urn:adsk.eagle:package:23682/2" value="100n"/>
@@
 <part name="R2A" library="rcl" library_urn="urn:adsk.eagle:library:334" deviceset="R-EU_" device="R1206" package3d_urn="urn:adsk.eagle:package:23540/2" value="750k"/>
 <part name="R2B" library="rcl" library_urn="urn:adsk.eagle:library:334" deviceset="R-EU_" device="R1206" package3d_urn="urn:adsk.eagle:package:23540/2" value="750k"/>
+<part name="C2" library="rcl" library_urn="urn:adsk.eagle:library:334" deviceset="C-EU" device="C1206K" package3d_urn="urn:adsk.eagle:package:23682/2" value="100n"/>
 </parts>
 <sheets>
@@
 <attribute name="VALUE" x="187.96" y="91.44" size="1.778" layer="96" rot="R180"/>
 </instance>
-<instance part="C1" gate="G$1" x="172.72" y="93.98" smashed="yes">
-<attribute name="NAME" x="173.863" y="94.4626" size="1.778" layer="95"/>
-<attribute name="VALUE" x="173.863" y="89.3826" size="1.778" layer="96"/>
-</instance>
-<instance part="GND8" gate="1" x="172.72" y="86.36" smashed="yes">
-<attribute name="VALUE" x="170.18" y="83.82" size="1.778" layer="96"/>
+<instance part="C1" gate="G$1" x="177.8" y="96.52" smashed="yes" rot="R270">
+<attribute name="NAME" x="178.2826" y="95.377" size="1.778" layer="95" rot="R270"/>
+<attribute name="VALUE" x="173.2026" y="95.377" size="1.778" layer="96" rot="R270"/>
+</instance>
+<instance part="GND8" gate="1" x="172.72" y="91.44" smashed="yes">
+<attribute name="VALUE" x="170.18" y="88.9" size="1.778" layer="96"/>
 </instance>
 <instance part="T1" gate="G$1" x="187.96" y="35.56" smashed="yes" rot="R270">
@@
 <attribute name="NAME" x="214.63" y="98.0186" size="1.778" layer="95"/>
 <attribute name="VALUE" x="214.63" y="93.218" size="1.778" layer="96"/>
+</instance>
+<instance part="C2" gate="G$1" x="170.18" y="48.26" smashed="yes">
+<attribute name="NAME" x="171.704" y="48.641" size="1.778" layer="95"/>
+<attribute name="VALUE" x="171.704" y="43.561" size="1.778" layer="96"/>
 </instance>
 </instances>
@@
 <wire x1="198.12" y1="43.18" x2="195.58" y2="43.18" width="0.1524" layer="91"/>
 <junction x="195.58" y="43.18"/>
+<pinref part="C2" gate="G$1" pin="2"/>
+<wire x1="170.18" y1="43.18" x2="180.34" y2="43.18" width="0.1524" layer="91"/>
 </segment>
 <segment>
@@
 <pinref part="C1" gate="G$1" pin="-"/>
 <pinref part="GND8" gate="1" pin="GND"/>
+<wire x1="172.72" y1="96.52" x2="172.72" y2="93.98" width="0.1524" layer="91"/>
 </segment>
 <segment>
@@
 <pinref part="IC5" gate="G$1" pin="V+"/>
 <pinref part="P+6" gate="VCC" pin="VCC"/>
+<pinref part="C2" gate="G$1" pin="1"/>
+<wire x1="170.18" y1="50.8" x2="170.18" y2="86.36" width="0.1524" layer="91"/>
+<wire x1="170.18" y1="86.36" x2="180.34" y2="86.36" width="0.1524" layer="91"/>
+<junction x="180.34" y="86.36"/>
 </segment>
 </net>
@@
 <junction x="180.34" y="96.52"/>
 <pinref part="C1" gate="G$1" pin="+"/>
-<wire x1="172.72" y1="96.52" x2="180.34" y2="96.52" width="0.1524" layer="91"/>
 <pinref part="P+4" gate="1" pin="V+"/>
 <wire x1="180.34" y1="101.6" x2="180.34" y2="96.52" width="0.1524" layer="91"/>
